File: portalhubkicad/portalhub.kicad_pcb (KiCad board)
At the start: 2 copper layers, 73.5 x 73.1 mm, 19 parts

Commit message: updated pcb and reuploaded
Parts:
- removed the CIN at (156.1, 124.7)
- removed the USBIN at (161.7, 130.5)
- added CIN: , portalhub-easyedapro:C0603, F.Cu at (156.1, 124.7)
- added USBIN: , portalhub-easyedapro:USB-C-SMD_TYPE-C-16PIN-2MD-073, F.Cu at (161.7, 130.5)
- C1, C10, C2, C3, C4, C5, C6, C7, C8, C9: footprint portalusbh-easyedapro:C0603 -> portalhub-easyedapro:C0603
- R1, R2: footprint portalusbh-easyedapro:R0603 -> portalhub-easyedapro:R0603
- U1: footprint portalusbh-easyedapro:SSOP-16_L4.6-W2.6-P0.53-LS4.0-BL -> portalhub-easyedapro:SSOP-16_L4.6-W2.6-P0.53-LS4.0-BL
- USB1, USB2, USB3, USB4: footprint portalusbh-easyedapro:USB-A-TH_10.0QHHTZB6.3 -> portalhub-easyedapro:USB-A-TH_10.0QHHTZB6.3
