File: portalhubkicad/portalhub.kicad_sch (KiCad schematic)
At the start: 20 parts, among them U1 SL2.1s

Commit message: updated pcb and reuploaded
Parts:
- removed ?: (no value), portalusbh-easyedapro:, symbol portalusbh-easyedapro:Drawing-Symbol_A4
- removed C1, C10, C2, C3, C4, C5, C6, C7, C8, C9, CIN: 100nF, portalusbh-easyedapro:C0603, symbol portalusbh-easyedapro:CAP
- removed R1, R2: 10K, portalusbh-easyedapro:R0603, symbol portalusbh-easyedapro:Res
- removed U1: SL2.1s, portalusbh-easyedapro:SSOP-16_L4.6-W2.6-P0.53-LS4.0-BL, symbol portalusbh-easyedapro:SL2.1S
- removed USB1, USB2, USB3, USB4: 10.0 QHHTZB6.3, portalusbh-easyedapro:USB-A-TH_10.0QHHTZB6.3, symbol portalusbh-easyedapro:10.0 QHHTZB6.3
- removed USBIN: TYPE-C 16PIN 2MD(073), portalusbh-easyedapro:USB-C-SMD_TYPE-C-16PIN-2MD-073, symbol portalusbh-easyedapro:TYPE-C 16PIN 2MD(073)
- added ?: (no value), portalhub-easyedapro:, symbol portalhub-easyedapro:Drawing-Symbol_A4
- added C1, C10, C2, C3, C4, C5, C6, C7, C8, C9, CIN: 100nF, portalhub-easyedapro:C0603, symbol portalhub-easyedapro:CAP
- added R1, R2: 10K, portalhub-easyedapro:R0603, symbol portalhub-easyedapro:Res
- added U1: SL2.1s, portalhub-easyedapro:SSOP-16_L4.6-W2.6-P0.53-LS4.0-BL, symbol portalhub-easyedapro:SL2.1S
- added USB1, USB2, USB3, USB4: 10.0 QHHTZB6.3, portalhub-easyedapro:USB-A-TH_10.0QHHTZB6.3, symbol portalhub-easyedapro:10.0 QHHTZB6.3
- added USBIN: TYPE-C 16PIN 2MD(073), portalhub-easyedapro:USB-C-SMD_TYPE-C-16PIN-2MD-073, symbol portalhub-easyedapro:TYPE-C 16PIN 2MD(073)
Connections:
- net +5V: now also C1.1, C2.1, C3.1, C4.1, C5.1, C6.1, CIN.1, U1.7 (VDD5), USB1.1 (VCC), USB2.1 (VCC), USB3.1 (VCC), USB4.1 (VCC), USBIN.A4B9 (VBUS), USBIN.B4A9 (VBUS)
- net DN: now also U1.5 (UDM), USBIN.A7 (Dn1), USBIN.B7 (Dn2)
- net DN1: now also U1.3 (DM1), USB1.2 (D-)
- net DN2: now also U1.1 (DM2), USB2.2 (D-)
- net DN3: now also U1.15 (DM3), USB3.2 (D-)
- net DN4: now also U1.13 (DM4), USB4.2 (D-)
- net DP: now also U1.6 (UDP), USBIN.A6 (Dp1), USBIN.B6 (Dp2)
- net DP1: now also U1.4 (DP1), USB1.3 (D+)
- net DP2: now also U1.2 (DP2), USB2.3 (D+)
- net DP3: now also U1.16 (DP3), USB3.3 (D+)
- net DP4: now also U1.14 (DP4), USB4.3 (D+)
- net GND: now also C1.2, C10.2, C2.2, C3.2, C4.2, C5.2, C6.2, C7.2, C8.2, C9.2, CIN.2, R1.1, R2.1, U1.12 (XIN), U1.8 (VSS), USB1.4 (GND), USB1.5, USB1.6, USB2.4 (GND), USB2.5, USB2.6, USB3.4 (GND), USB3.5, USB3.6, USB4.4 (GND), USB4.5, USB4.6, USBIN.13 (EH), USBIN.14 (EH), USBIN.A1B12 (GND), USBIN.B1A12 (GND)
- new net: C10.1, C9.1, U1.10 (VDD18)
- new net: C7.1, C8.1, U1.9 (VDD33)
- new net: R1.2, USBIN.A5 (CC1)
- new net: R2.2, USBIN.B5 (CC2)
